File: kicad/kitbashkvm-protoboard/kitbashkvm-protoboard.kicad_sch (KiCad schematic)
At the start: 0 parts

Commit message: kicad files and updated gitignore
Parts:
- added CH9329: ~, breakout-components:CH9329_UART_TO_USB_2.0, symbol breakout-components:CH9329_UART_TO_USB_2.0
- added USB_2.0_HUB1: ~, breakout-components:USB_2.0_HUB, symbol breakout-components:USB_2.0_HUB
- added USB_A_2.0_F1: ~, breakout-components:USB_A_2.0_F, symbol breakout-components:USB_A_2.0_F
- added USB_C_2.0_F1, USB_C_2.0_F2: ~, breakout-components:USB_C_2.0_F, symbol breakout-components:USB_C_2.0_F
- added USB_SER1: ~, breakout-components:CH340_TO_USB_2.0, symbol breakout-components:CH340_TO_USB_2.0
Connections:
- new net: CH9329.1 (5v), USB_C_2.0_F1.1 (VBUS)
- new net: CH9329.4 (GND), USB_C_2.0_F1.2 (GND)
- new net: CH9329.2 (D-), USB_C_2.0_F1.4 (D-)
- new net: CH9329.3 (D+), USB_C_2.0_F1.5 (D+)
- new net: USB_2.0_HUB1.13 (GND), USB_A_2.0_F1.1 (GND)
- new net: USB_2.0_HUB1.14 (D+), USB_A_2.0_F1.2 (D+)
- new net: USB_2.0_HUB1.15 (D-), USB_A_2.0_F1.3 (D-)
- new net: USB_2.0_HUB1.16 (5v), USB_A_2.0_F1.4 (VBUS)
- new net: CH9329.6 (TX), USB_SER1.2 (RX)
- new net: CH9329.7 (RX), USB_SER1.3 (TX)
- new net: CH9329.8 (GND), USB_SER1.1 (GND)
- new net: USB_2.0_HUB1.5 (GND), USB_SER1.5 (GND)
- new net: USB_2.0_HUB1.6 (D+), USB_SER1.6 (D+)
- new net: USB_2.0_HUB1.7 (D-), USB_SER1.7 (D-)
- new net: USB_2.0_HUB1.8 (5v), USB_SER1.8 (5v)
- new net: USB_2.0_HUB1.10 (D+), USB_C_2.0_F2.5 (D+)
- new net: USB_2.0_HUB1.11 (D-), USB_C_2.0_F2.4 (D-)
- new net: USB_2.0_HUB1.12 (5v), USB_C_2.0_F2.1 (VBUS)
- new net: USB_2.0_HUB1.9 (GND), USB_C_2.0_F2.2 (GND)
